Commit message: Corrected joint orientation

File: body.urdf (robot description, URDF)
Before this commit: robot robot, 3 links, 2 joints
Joints:
- joint BackLeg_Torso: origin xyz=0 0.5 1 rpy=0 0 0 -> xyz=0.5 0 1 rpy=0 0 0
- joint Torso_FrontLeg: origin xyz=0 1 0 rpy=0 0 0 -> xyz=1 0 0 rpy=0 0 0

Commit message: Finished Task N

File: body.urdf (robot description, URDF)
Before this commit: robot robot, 3 links, 2 joints
Links:
- added link BackLowerLeg, mass 1; collision box size=0.2 0.2 1; visual box size=0.2 0.2 1
- added link FrontLowerLeg, mass 1; collision box size=0.2 0.2 1; visual box size=0.2 0.2 1
- added link LeftLeg, mass 1; collision box size=1.0 0.2 0.2; visual box size=1.0 0.2 0.2
- added link LeftLowerLeg, mass 1; collision box size=0.2 0.2 1; visual box size=0.2 0.2 1
- added link RightLeg, mass 1; collision box size=1 0.2 0.2; visual box size=1 0.2 0.2
- added link RightLowerLeg, mass 1; collision box size=0.2 0.2 1; visual box size=0.2 0.2 1
- link BackLeg: geometry collision box size=0.2 1 0.2; visual box size=0.2 1 0.2
- link FrontLeg: geometry collision box size=0.2 1 0.2; visual box size=0.2 1 0.2
Joints:
- added joint BackLeg_BackLowerLeg: type revolute, parent BackLeg, child BackLowerLeg, origin xyz=0 -1 0 rpy=0 0 0, axis 1 0 0, limit lower=-3.14159 upper=3.14159 effort=0.0 velocity=0.0
- added joint FrontLeg_FrontLowerLeg: type revolute, parent FrontLeg, child FrontLowerLeg, origin xyz=0 1 0 rpy=0 0 0, axis 1 0 0, limit lower=-3.14159 upper=3.14159 effort=0.0 velocity=0.0
- added joint LeftLeg_LeftLowerLeg: type revolute, parent LeftLeg, child LeftLowerLeg, origin xyz=-1 0 0 rpy=0 0 0, axis 0 1 0, limit lower=-3.14159 upper=3.14159 effort=0.0 velocity=0.0
- added joint RightLeg_RightLowerLeg: type revolute, parent RightLeg, child RightLowerLeg, origin xyz=1 0 0 rpy=0 0 0, axis 0 1 0, limit lower=-3.14159 upper=3.14159 effort=0.0 velocity=0.0
- added joint Torso_LeftLeg: type revolute, parent Torso, child LeftLeg, origin xyz=-0.5 0 1 rpy=0 0 0, axis 0 1 0, limit lower=-3.14159 upper=3.14159 effort=0.0 velocity=0.0
- added joint Torso_RightLeg: type revolute, parent Torso, child RightLeg, origin xyz=0.5 0 1 rpy=0 0 0, axis 0 1 0, limit lower=-3.14159 upper=3.14159 effort=0.0 velocity=0.0
- joint Torso_BackLeg: axis 0 1 0 -> 1 0 0; origin xyz=1 0 1 rpy=0 0 0 -> xyz=0 -0.5 1 rpy=0 0 0
- joint Torso_FrontLeg: axis 0 1 0 -> 1 0 0; origin xyz=2 0 1 rpy=0 0 0 -> xyz=0 0.5 1 rpy=0 0 0

Commit message: Submission for Assign. 5

File: body.urdf (robot description, URDF)
Before this commit: robot robot, 9 links, 8 joints
Links:
- removed link BackLeg
- removed link BackLowerLeg
- removed link FrontLeg
- removed link FrontLowerLeg
- removed link LeftLeg
- removed link LeftLowerLeg
- removed link RightLeg
- removed link RightLowerLeg
- added link BackLeftLeg, mass 1; collision box size=0.1 0.1 1; visual box size=0.1 0.1 1
- added link BackRightLeg, mass 1; collision box size=0.1 0.1 1; visual box size=0.1 0.1 1
- added link FrontLeftLeg, mass 1; collision box size=0.1 0.1 1; visual box size=0.1 0.1 1
- added link FrontRightLeg, mass 1; collision box size=0.1 0.1 1; visual box size=0.1 0.1 1
- added link Head, mass 1; collision box size=0.3 0.2 0.2; visual box size=0.3 0.2 0.2
- added link Tail, mass 1; collision box size=0.8 0.1 0.1; visual box size=0.8 0.1 0.1
- link Torso: geometry collision box size=1 0.5 0.2; visual box size=1 0.5 0.2
Joints:
- removed joint BackLeg_BackLowerLeg
- removed joint FrontLeg_FrontLowerLeg
- removed joint LeftLeg_LeftLowerLeg
- removed joint RightLeg_RightLowerLeg
- removed joint Torso_BackLeg
- removed joint Torso_FrontLeg
- removed joint Torso_LeftLeg
- removed joint Torso_RightLeg
- added joint Torso_BackLeftLeg: type revolute, parent Torso, child BackLeftLeg, origin xyz=0.5 -0.1 1 rpy=0 0 0, axis 0 1 0, limit lower=-3.14159 upper=3.14159 effort=0.0 velocity=0.0
- added joint Torso_BackRightLeg: type revolute, parent Torso, child BackRightLeg, origin xyz=0.5 0.1 1 rpy=0 0 0, axis 0 1 0, limit lower=-3.14159 upper=3.14159 effort=0.0 velocity=0.0
- added joint Torso_FrontLeftLeg: type revolute, parent Torso, child FrontLeftLeg, origin xyz=-0.5 -0.1 1 rpy=0 0 0, axis 0 1 0, limit lower=-3.14159 upper=3.14159 effort=0.0 velocity=0.0
- added joint Torso_FrontRightLeg: type revolute, parent Torso, child FrontRightLeg, origin xyz=-0.5 0.1 1 rpy=0 0 0, axis 0 1 0, limit lower=-3.14159 upper=3.14159 effort=0.0 velocity=0.0
- added joint Torso_Head: type revolute, parent Torso, child Head, origin xyz=-0.5 0 1 rpy=0 0 0, axis 1 0 0, limit lower=-3.14159 upper=3.14159 effort=0.0 velocity=0.0
- added joint Torso_Tail: type revolute, parent Torso, child Tail, origin xyz=0.5 0 1 rpy=0 0 0, axis 0 1 0, limit lower=-3.14159 upper=3.14159 effort=0.0 velocity=0.0

Commit message: Snakes first commit

File: body.urdf (robot description, URDF)
Before this commit: robot robot, 7 links, 6 joints
Links:
- removed link BackLeftLeg
- removed link BackRightLeg
- removed link FrontLeftLeg
- removed link FrontRightLeg
- removed link Head
- removed link Tail
- removed link Torso
- added link 0, mass 1; collision box size=0.42484415634250816 0.4518508959884525 0.46576951599868494; visual box size=0.42484415634250816 0.4518508959884525 0.46576951599868494
- added link 1, mass 1; collision box size=0.4836574057049045 0.4356432363394632 0.49509193629955073; visual box size=0.4836574057049045 0.4356432363394632 0.49509193629955073
- added link 10, mass 1; collision box size=0.2660500523622125 0.3722588918294921 0.3882505644145581; visual box size=0.2660500523622125 0.3722588918294921 0.3882505644145581
- added link 11, mass 1; collision box size=0.25975510714489697 0.4722087228636733 0.22019273249347135; visual box size=0.25975510714489697 0.4722087228636733 0.22019273249347135
- added link 12, mass 1; collision box size=0.2768593314771188 0.46442769701124054 0.2023956082146997; visual box size=0.2768593314771188 0.46442769701124054 0.2023956082146997
- added link 13, mass 1; collision box size=0.24903947495369594 0.2258182171066387 0.40154626092744117; visual box size=0.24903947495369594 0.2258182171066387 0.40154626092744117
- added link 14, mass 1; collision box size=0.24109106089283927 0.277951567731852 0.4850696967822896; visual box size=0.24109106089283927 0.277951567731852 0.4850696967822896
- added link 15, mass 1; collision box size=0.25213379411779163 0.48923632588220384 0.4751637347781806; visual box size=0.25213379411779163 0.48923632588220384 0.4751637347781806
- added link 16, mass 1; collision box size=0.3864848808187319 0.45234227371170893 0.3825539464782298; visual box size=0.3864848808187319 0.45234227371170893 0.3825539464782298
- added link 2, mass 1; collision box size=0.2481737628917602 0.4423867925594138 0.41398664745575736; visual box size=0.2481737628917602 0.4423867925594138 0.41398664745575736
- added link 3, mass 1; collision box size=0.49285160765967706 0.2459085430090778 0.2840659230202233; visual box size=0.49285160765967706 0.2459085430090778 0.2840659230202233
- added link 4, mass 1; collision box size=0.37542502020343427 0.2512809971530779 0.2589947487124105; visual box size=0.37542502020343427 0.2512809971530779 0.2589947487124105
- added link 5, mass 1; collision box size=0.4516005417023585 0.48322034688125964 0.3281368339620758; visual box size=0.4516005417023585 0.48322034688125964 0.3281368339620758
- added link 6, mass 1; collision box size=0.33951410421122863 0.3098771348162262 0.20779329478373199; visual box size=0.33951410421122863 0.3098771348162262 0.20779329478373199
- added link 7, mass 1; collision box size=0.2608980659914087 0.4498001986414032 0.2519673636576072; visual box size=0.2608980659914087 0.4498001986414032 0.2519673636576072
- added link 8, mass 1; collision box size=0.2774919645810685 0.315308510187129 0.27215037554367794; visual box size=0.2774919645810685 0.315308510187129 0.27215037554367794
- added link 9, mass 1; collision box size=0.44817501585082165 0.34397894932836415 0.30083258942186314; visual box size=0.44817501585082165 0.34397894932836415 0.30083258942186314
Joints:
- removed joint Torso_BackLeftLeg
- removed joint Torso_BackRightLeg
- removed joint Torso_FrontLeftLeg
- removed joint Torso_FrontRightLeg
- removed joint Torso_Head
- removed joint Torso_Tail
- added joint 0_1: type revolute, parent 0, child 1, origin xyz=0.21242207817125408 0 1 rpy=0 0 0, axis 0 0 1, limit lower=-3.14159 upper=3.14159 effort=0.0 velocity=0.0
- added joint 10_11: type revolute, parent 10, child 11, origin xyz=1.954943796760544 0 1 rpy=0 0 0, axis 0 0 1, limit lower=-3.14159 upper=3.14159 effort=0.0 velocity=0.0
- added joint 11_12: type revolute, parent 11, child 12, origin xyz=2.081673877724335 0 1 rpy=0 0 0, axis 0 0 1, limit lower=-3.14159 upper=3.14159 effort=0.0 velocity=0.0
- added joint 12_13: type revolute, parent 12, child 13, origin xyz=2.228655655629005 0 1 rpy=0 0 0, axis 0 0 1, limit lower=-3.14159 upper=3.14159 effort=0.0 velocity=0.0
- added joint 13_14: type revolute, parent 13, child 14, origin xyz=2.3392654648441416 0 1 rpy=0 0 0, axis 0 0 1, limit lower=-3.14159 upper=3.14159 effort=0.0 velocity=0.0
- added joint 14_15: type revolute, parent 14, child 15, origin xyz=2.455836788260133 0 1 rpy=0 0 0, axis 0 0 1, limit lower=-3.14159 upper=3.14159 effort=0.0 velocity=0.0
- added joint 15_16: type revolute, parent 15, child 16, origin xyz=2.587425051931505 0 1 rpy=0 0 0, axis 0 0 1, limit lower=-3.14159 upper=3.14159 effort=0.0 velocity=0.0
- added joint 1_2: type revolute, parent 1, child 2, origin xyz=0.4836574057049045 0 1 rpy=0 0 0, axis 0 0 1, limit lower=-3.14159 upper=3.14159 effort=0.0 velocity=0.0
- added joint 2_3: type revolute, parent 2, child 3, origin xyz=0.49000246574421247 0 1 rpy=0 0 0, axis 0 0 1, limit lower=-3.14159 upper=3.14159 effort=0.0 velocity=0.0
- added joint 3_4: type revolute, parent 3, child 4, origin xyz=0.8587671919580095 0 1 rpy=0 0 0, axis 0 0 1, limit lower=-3.14159 upper=3.14159 effort=0.0 velocity=0.0
- added joint 4_5: type revolute, parent 4, child 5, origin xyz=0.9877664083316053 0 1 rpy=0 0 0, axis 0 0 1, limit lower=-3.14159 upper=3.14159 effort=0.0 velocity=0.0
- added joint 5_6: type revolute, parent 5, child 6, origin xyz=1.2516544399322467 0 1 rpy=0 0 0, axis 0 0 1, limit lower=-3.14159 upper=3.14159 effort=0.0 velocity=0.0
- added joint 6_7: type revolute, parent 6, child 7, origin xyz=1.365368273292296 0 1 rpy=0 0 0, axis 0 0 1, limit lower=-3.14159 upper=3.14159 effort=0.0 velocity=0.0
- added joint 7_8: type revolute, parent 7, child 8, origin xyz=1.4565092871780907 0 1 rpy=0 0 0, axis 0 0 1, limit lower=-3.14159 upper=3.14159 effort=0.0 velocity=0.0
- added joint 8_9: type revolute, parent 8, child 9, origin xyz=1.603552218763455 0 1 rpy=0 0 0, axis 0 0 1, limit lower=-3.14159 upper=3.14159 effort=0.0 velocity=0.0
- added joint 9_10: type revolute, parent 9, child 10, origin xyz=1.9129812523237422 0 1 rpy=0 0 0, axis 0 0 1, limit lower=-3.14159 upper=3.14159 effort=0.0 velocity=0.0

Commit message: Before finishing snakes

File: body.urdf (robot description, URDF)
Before this commit: robot robot, 17 links, 16 joints
Links:
- removed link 10
- removed link 11
- removed link 12
- removed link 13
- removed link 14
- removed link 15
- removed link 16
- removed link 2
- removed link 3
- removed link 4
- removed link 5
- removed link 6
- removed link 7
- removed link 8
- removed link 9
- link 0: geometry collision box size=0.31834394140045236 0.3015427063526149 0.2155169198741038; visual box size=0.31834394140045236 0.3015427063526149 0.2155169198741038
- link 1: geometry collision box size=0.2739670298059541 0.2542088209786305 0.27354106128265665; visual box size=0.2739670298059541 0.2542088209786305 0.27354106128265665
Joints:
- removed joint 10_11
- removed joint 11_12
- removed joint 12_13
- removed joint 13_14
- removed joint 14_15
- removed joint 15_16
- removed joint 1_2
- removed joint 2_3
- removed joint 3_4
- removed joint 4_5
- removed joint 5_6
- removed joint 6_7
- removed joint 7_8
- removed joint 8_9
- removed joint 9_10
- joint 0_1: origin xyz=0.21242207817125408 0 1 rpy=0 0 0 -> xyz=0.15917197070022618 0 1 rpy=0 0 0

Commit message: snakes 2

File: body.urdf (robot description, URDF)
Before this commit: robot robot, 2 links, 1 joints
Links:
- added link 10, mass 1; collision box size=0.48595196754625974 0.3263141215821568 0.47403240554068893; visual box size=0.48595196754625974 0.3263141215821568 0.47403240554068893
- added link 11, mass 1; collision box size=0.27337515000147466 0.21063668645505015 0.38862356569086864; visual box size=0.27337515000147466 0.21063668645505015 0.38862356569086864
- added link 2, mass 1; collision box size=0.4984051218186364 0.49352582493244446 0.4650746748944219; visual box size=0.4984051218186364 0.49352582493244446 0.4650746748944219
- added link 3, mass 1; collision box size=0.28715159497022413 0.48387240425630834 0.49803100516563825; visual box size=0.28715159497022413 0.48387240425630834 0.49803100516563825
- added link 4, mass 1; collision box size=0.21084588236864144 0.24820366287626983 0.3125713887217378; visual box size=0.21084588236864144 0.24820366287626983 0.3125713887217378
- added link 5, mass 1; collision box size=0.30718578703476723 0.3457202358248612 0.4008180222452664; visual box size=0.30718578703476723 0.3457202358248612 0.4008180222452664
- added link 6, mass 1; collision box size=0.3858999868774605 0.3889634948027241 0.4612764158429726; visual box size=0.3858999868774605 0.3889634948027241 0.4612764158429726
- added link 7, mass 1; collision box size=0.48752155194619345 0.30638952433994043 0.36443506262435255; visual box size=0.48752155194619345 0.30638952433994043 0.36443506262435255
- added link 8, mass 1; collision box size=0.478712296549656 0.3203940303793281 0.4906223252555815; visual box size=0.478712296549656 0.3203940303793281 0.4906223252555815
- added link 9, mass 1; collision box size=0.4109551293792979 0.30968325739142116 0.49366853730643734; visual box size=0.4109551293792979 0.30968325739142116 0.49366853730643734
- link 0: geometry collision box size=0.6 0.6 0.6; visual box size=0.6 0.6 0.6
- link 1: geometry collision box size=0.3930962158164426 0.41273271717387505 0.3583813728731955; visual box size=0.3930962158164426 0.41273271717387505 0.3583813728731955
Joints:
- added joint 10_11: type revolute, parent 10, child 11, origin xyz=0.48595196754625974 0 0 rpy=0 0 0, axis 0 0 1, limit lower=-3.14159 upper=3.14159 effort=0.0 velocity=0.0
- added joint 1_2: type revolute, parent 1, child 2, origin xyz=0.3930962158164426 0 0 rpy=0 0 0, axis 0 0 1, limit lower=-3.14159 upper=3.14159 effort=0.0 velocity=0.0
- added joint 2_3: type revolute, parent 2, child 3, origin xyz=0.4984051218186364 0 0 rpy=0 0 0, axis 0 0 1, limit lower=-3.14159 upper=3.14159 effort=0.0 velocity=0.0
- added joint 3_4: type revolute, parent 3, child 4, origin xyz=0.28715159497022413 0 0 rpy=0 0 0, axis 0 0 1, limit lower=-3.14159 upper=3.14159 effort=0.0 velocity=0.0
- added joint 4_5: type revolute, parent 4, child 5, origin xyz=0.21084588236864144 0 0 rpy=0 0 0, axis 0 0 1, limit lower=-3.14159 upper=3.14159 effort=0.0 velocity=0.0
- added joint 5_6: type revolute, parent 5, child 6, origin xyz=0.30718578703476723 0 0 rpy=0 0 0, axis 0 0 1, limit lower=-3.14159 upper=3.14159 effort=0.0 velocity=0.0
- added joint 6_7: type revolute, parent 6, child 7, origin xyz=0.3858999868774605 0 0 rpy=0 0 0, axis 0 0 1, limit lower=-3.14159 upper=3.14159 effort=0.0 velocity=0.0
- added joint 7_8: type revolute, parent 7, child 8, origin xyz=0.48752155194619345 0 0 rpy=0 0 0, axis 0 0 1, limit lower=-3.14159 upper=3.14159 effort=0.0 velocity=0.0
- added joint 8_9: type revolute, parent 8, child 9, origin xyz=0.478712296549656 0 0 rpy=0 0 0, axis 0 0 1, limit lower=-3.14159 upper=3.14159 effort=0.0 velocity=0.0
- added joint 9_10: type revolute, parent 9, child 10, origin xyz=0.4109551293792979 0 0 rpy=0 0 0, axis 0 0 1, limit lower=-3.14159 upper=3.14159 effort=0.0 velocity=0.0
- joint 0_1: origin xyz=0.15917197070022618 0 1 rpy=0 0 0 -> xyz=0.3 0 0.15 rpy=0 0 0

Commit message: finished snakes

File: body.urdf (robot description, URDF)
Before this commit: robot robot, 12 links, 11 joints
Links:
- removed link 11
- link 1: geometry collision box size=0.40001420966123535 0.4236418122444947 0.44886334802902245; visual box size=0.40001420966123535 0.4236418122444947 0.44886334802902245
- link 10: geometry collision box size=0.28835381049386377 0.347582013423615 0.40722963975590865; visual box size=0.28835381049386377 0.347582013423615 0.40722963975590865
- link 2: geometry collision box size=0.36277354478657 0.35461146818058487 0.4973179719598263; visual box size=0.36277354478657 0.35461146818058487 0.4973179719598263
- link 3: geometry collision box size=0.44003868703024507 0.3658024997611757 0.4541731207231018; visual box size=0.44003868703024507 0.3658024997611757 0.4541731207231018
- link 4: geometry collision box size=0.21553528660201562 0.4553122546093196 0.36684105225388974; visual box size=0.21553528660201562 0.4553122546093196 0.36684105225388974
- link 5: geometry collision box size=0.2635296712400413 0.21226923869325337 0.36313830082366005; visual box size=0.2635296712400413 0.21226923869325337 0.36313830082366005
- link 6: geometry collision box size=0.3024046795181018 0.3683704924127811 0.37872552272528404; visual box size=0.3024046795181018 0.3683704924127811 0.37872552272528404
- link 7: geometry collision box size=0.3974250163059375 0.3469477876691793 0.38317136533736107; visual box size=0.3974250163059375 0.3469477876691793 0.38317136533736107
- link 8: geometry collision box size=0.23198366132207604 0.2257828877026843 0.361295756821446; visual box size=0.23198366132207604 0.2257828877026843 0.361295756821446
- link 9: geometry collision box size=0.47421250137334725 0.4799260068209846 0.29392715711504575; visual box size=0.47421250137334725 0.4799260068209846 0.29392715711504575
Joints:
- removed joint 10_11
- joint 0_1: origin xyz=0.3 0 0.15 rpy=0 0 0 -> xyz=0.3 0 0.25 rpy=0 0 0
- joint 1_2: axis 0 0 1 -> 0 1 0; origin xyz=0.3930962158164426 0 0 rpy=0 0 0 -> xyz=0.40001420966123535 0 0 rpy=0 0 0
- joint 2_3: axis 0 0 1 -> 0 1 0; origin xyz=0.4984051218186364 0 0 rpy=0 0 0 -> xyz=0.36277354478657 0 0 rpy=0 0 0
- joint 3_4: axis 0 0 1 -> 0 1 0; origin xyz=0.28715159497022413 0 0 rpy=0 0 0 -> xyz=0.44003868703024507 0 0 rpy=0 0 0
- joint 4_5: origin xyz=0.21084588236864144 0 0 rpy=0 0 0 -> xyz=0.21553528660201562 0 0 rpy=0 0 0
- joint 5_6: origin xyz=0.30718578703476723 0 0 rpy=0 0 0 -> xyz=0.2635296712400413 0 0 rpy=0 0 0
- joint 6_7: axis 0 0 1 -> 0 1 0; origin xyz=0.3858999868774605 0 0 rpy=0 0 0 -> xyz=0.3024046795181018 0 0 rpy=0 0 0
- joint 7_8: origin xyz=0.48752155194619345 0 0 rpy=0 0 0 -> xyz=0.3974250163059375 0 0 rpy=0 0 0
- joint 8_9: axis 0 0 1 -> 0 1 0; origin xyz=0.478712296549656 0 0 rpy=0 0 0 -> xyz=0.23198366132207604 0 0 rpy=0 0 0
- joint 9_10: origin xyz=0.4109551293792979 0 0 rpy=0 0 0 -> xyz=0.47421250137334725 0 0 rpy=0 0 0

Commit message: Finished assign. 7

File: body.urdf (robot description, URDF)
Before this commit: robot robot, 8 links, 7 joints
Links:
- added link 8, mass 1; collision box size=0.30823807179156726 0.348382860064279 0.2673784255821975; visual box size=0.30823807179156726 0.348382860064279 0.2673784255821975
- added link 9, mass 1; collision box size=0.3342088379291028 0.23160864786220567 0.2803392531874344; visual box size=0.3342088379291028 0.23160864786220567 0.2803392531874344
- link 1: geometry collision box size=0.49179642403193635 0.24600726369235418 0.4467946856675866; visual box size=0.49179642403193635 0.24600726369235418 0.4467946856675866
- link 2: geometry collision box size=0.21407666270525028 0.33795136050528424 0.3395545129987635; visual box size=0.21407666270525028 0.33795136050528424 0.3395545129987635
- link 3: geometry collision box size=0.31393407544856144 0.2162431753862355 0.37895498814160844; visual box size=0.31393407544856144 0.2162431753862355 0.37895498814160844
- link 4: geometry collision box size=0.2984632792671199 0.4059385241869412 0.26153961498693856; visual box size=0.2984632792671199 0.4059385241869412 0.26153961498693856
- link 5: geometry collision box size=0.303388521957081 0.2023678552467354 0.3782461912424998; visual box size=0.303388521957081 0.2023678552467354 0.3782461912424998
- link 6: geometry collision box size=0.5508134799756204 0.34000540349401864 0.26811288230132035; visual box size=0.5508134799756204 0.34000540349401864 0.26811288230132035
- link 7: geometry collision box size=0.569243732673813 0.21765635735728986 0.331924472454202; visual box size=0.569243732673813 0.21765635735728986 0.331924472454202
Joints:
- added joint 7_8: type revolute, parent 7, child 8, origin xyz=0.0 0.10882817867864493 -0.1891230956212499 rpy=0 0 0, axis 0 0 1, limit lower=-3.14159 upper=3.14159 effort=0.0 velocity=0.0
- added joint 8_9: type revolute, parent 8, child 9, origin xyz=0.0 -0.10882817867864493 -0.13368921279109874 rpy=0 0 0, axis 0 0 1, limit lower=-3.14159 upper=3.14159 effort=0.0 velocity=0.0
- joint 1_2: axis 0 1 0 -> 0 0 1; origin xyz=0 -0.38482667985487595 0 rpy=0 0 0 -> xyz=0.2 0 0.25 rpy=0 0 0
- joint 2_3: axis 0 1 0 -> 0 0 1; origin xyz=0.40755530531766526 0 0 rpy=0 0 0 -> xyz=0.0 0.16897568025264212 -0.25 rpy=0 0 0
- joint 3_4: axis 0 1 0 -> 0 0 1; origin xyz=0 0 -0.3878040172221531 rpy=0 0 0 -> xyz=0.15696703772428072 -0.16897568025264212 0.0 rpy=0 0 0
- joint 4_5: origin xyz=0 -0.3476509418914583 0 rpy=0 0 0 -> xyz=-0.15696703772428072 0.2029692620934706 0.0 rpy=0 0 0
- joint 5_6: origin xyz=-0.26100136936729956 0 0 rpy=0 0 0 -> xyz=0.0 -0.2029692620934706 0.1891230956212499 rpy=0 0 0
- joint 6_7: axis 1 0 0 -> 0 0 1; origin xyz=0 -0.4335901209472173 0 rpy=0 0 0 -> xyz=0.0 -0.2029692620934706 0.1891230956212499 rpy=0 0 0
