Commit message: Currently struggling

File: body.urdf (robot description, URDF)
Before this commit: robot robot, 3 links, 2 joints
Links:
- removed link BackLeg
- removed link FrontLeg
- removed link Torso
- added link 00, mass 1; collision box size=0.4 0.4 0.4; visual box size=0.4 0.4 0.4
- added link 01, mass 1; collision box size=0.2345242823893864 0.3071260350193112 0.28243462957826565; visual box size=0.2345242823893864 0.3071260350193112 0.28243462957826565
- added link 10, mass 1; collision box size=0.30589631530482764 0.3596609759677495 0.22999019163778522; visual box size=0.30589631530482764 0.3596609759677495 0.22999019163778522
- added link 11, mass 1; collision box size=0.31980837374190807 0.3605006216995754 0.37674278711716397; visual box size=0.31980837374190807 0.3605006216995754 0.37674278711716397
- added link 12, mass 1; collision box size=0.2940607787807493 0.3782707143681631 0.23059526124653507; visual box size=0.2940607787807493 0.3782707143681631 0.23059526124653507
- added link 13, mass 1; collision box size=0.30789407080155506 0.37611785826277744 0.3528412933417431; visual box size=0.30789407080155506 0.37611785826277744 0.3528412933417431
- added link 14, mass 1; collision box size=0.3218009141744317 0.3853797267501953 0.2401510219908636; visual box size=0.3218009141744317 0.3853797267501953 0.2401510219908636
- added link 15, mass 1; collision box size=0.2187343738358072 0.3430611698546724 0.211456369985951; visual box size=0.2187343738358072 0.3430611698546724 0.211456369985951
- added link 2, mass 1; collision box size=0.3552341902247608 0.32969302883118845 0.20973039820437425; visual box size=0.3552341902247608 0.32969302883118845 0.20973039820437425
- added link 3, mass 1; collision box size=0.39664161291638556 0.32245706205575275 0.33812803781622325; visual box size=0.39664161291638556 0.32245706205575275 0.33812803781622325
- added link 4, mass 1; collision box size=0.33134525618054533 0.2298506476176344 0.38462709616827706; visual box size=0.33134525618054533 0.2298506476176344 0.38462709616827706
- added link 5, mass 1; collision box size=0.36519194872504834 0.323858279874699 0.23895683394106693; visual box size=0.36519194872504834 0.323858279874699 0.23895683394106693
- added link 6, mass 1; collision box size=0.3886586716675638 0.29042303656814317 0.34656285972181766; visual box size=0.3886586716675638 0.29042303656814317 0.34656285972181766
- added link 7, mass 1; collision box size=0.23100510063857693 0.24182059259142968 0.39522852688044996; visual box size=0.23100510063857693 0.24182059259142968 0.39522852688044996
- added link 8, mass 1; collision box size=0.3437608037069486 0.23773875319915816 0.38871408268723723; visual box size=0.3437608037069486 0.23773875319915816 0.38871408268723723
- added link 9, mass 1; collision box size=0.23008053373087434 0.3137368890048676 0.2749031494231402; visual box size=0.23008053373087434 0.3137368890048676 0.2749031494231402
Joints:
- removed joint Torso_BackLeg
- removed joint Torso_FrontLeg
- added joint 00_1: type revolute, parent 0, child 1, origin xyz=0.2 0 0.5 rpy=0 0 0, axis 0 0 1, limit lower=-3.14159 upper=3.14159 effort=0.0 velocity=0.0
- added joint 10_11: type revolute, parent 10, child 11, origin xyz=0.267988424517851 0 0.0 rpy=0 0 0, axis 0 0 1, limit lower=-3.14159 upper=3.14159 effort=0.0 velocity=0.0
- added joint 11_12: type revolute, parent 11, child 12, origin xyz=-0.31285234452336785 0 0.0 rpy=0 0 0, axis 1 0 0, limit lower=-3.14159 upper=3.14159 effort=0.0 velocity=0.0
- added joint 12_13: type revolute, parent 12, child 13, origin xyz=0.3069345762613287 0 0.0 rpy=0 0 0, axis 0 1 0, limit lower=-3.14159 upper=3.14159 effort=0.0 velocity=0.0
- added joint 13_14: type revolute, parent 13, child 14, origin xyz=-0.3009774247911522 0 0.0 rpy=0 0 0, axis 0 0 1, limit lower=-3.14159 upper=3.14159 effort=0.0 velocity=0.0
- added joint 14_15: type revolute, parent 14, child 15, origin xyz=0.3148474924879934 0 0.0 rpy=0 0 0, axis 0 1 0, limit lower=-3.14159 upper=3.14159 effort=0.0 velocity=0.0
- added joint 1_2: type revolute, parent 1, child 2, origin xyz=-0.2 0 0.0 rpy=0 0 0, axis 1 0 0, limit lower=-3.14159 upper=3.14159 effort=0.0 velocity=0.0
- added joint 2_3: type revolute, parent 2, child 3, origin xyz=0.29487923630707363 0 0.0 rpy=0 0 0, axis 1 0 0, limit lower=-3.14159 upper=3.14159 effort=0.0 velocity=0.0
- added joint 3_4: type revolute, parent 3, child 4, origin xyz=-0.3759379015705732 0 0.0 rpy=0 0 0, axis 1 0 0, limit lower=-3.14159 upper=3.14159 effort=0.0 velocity=0.0
- added joint 4_5: type revolute, parent 4, child 5, origin xyz=0.36399343454846544 0 0.0 rpy=0 0 0, axis 1 0 0, limit lower=-3.14159 upper=3.14159 effort=0.0 velocity=0.0
- added joint 5_6: type revolute, parent 5, child 6, origin xyz=-0.34826860245279684 0 0.0 rpy=0 0 0, axis 0 1 0, limit lower=-3.14159 upper=3.14159 effort=0.0 velocity=0.0
- added joint 6_7: type revolute, parent 6, child 7, origin xyz=0.37692531019630604 0 0.0 rpy=0 0 0, axis 0 0 1, limit lower=-3.14159 upper=3.14159 effort=0.0 velocity=0.0
- added joint 7_8: type revolute, parent 7, child 8, origin xyz=-0.30983188615307033 0 0.0 rpy=0 0 0, axis 0 1 0, limit lower=-3.14159 upper=3.14159 effort=0.0 velocity=0.0
- added joint 8_9: type revolute, parent 8, child 9, origin xyz=0.2873829521727628 0 0.0 rpy=0 0 0, axis 0 0 1, limit lower=-3.14159 upper=3.14159 effort=0.0 velocity=0.0
- added joint 9_10: type revolute, parent 9, child 10, origin xyz=-0.2869206687189115 0 0.0 rpy=0 0 0, axis 0 1 0, limit lower=-3.14159 upper=3.14159 effort=0.0 velocity=0.0

Commit message: About to parallelize

File: body.urdf (robot description, URDF)
Before this commit: robot robot, 3 links, 2 joints
Links:
- removed link BackLeg
- removed link FrontLeg
- removed link Torso
- added link 0, mass 1; collision box size=0.4 0.4 0.4; visual box size=0.4 0.4 0.4
- added link 1, mass 1; collision box size=0.4925597713120326 0.26481633625635537 0.22909773036884534; visual box size=0.4925597713120326 0.26481633625635537 0.22909773036884534
- added link 2, mass 1; collision box size=0.21544209887787383 0.4793667442115083 0.4743572666951317; visual box size=0.21544209887787383 0.4793667442115083 0.4743572666951317
- added link 3, mass 1; collision box size=0.26267285158109266 0.4264517289799963 0.4421824630930003; visual box size=0.26267285158109266 0.4264517289799963 0.4421824630930003
- added link 4, mass 1; collision box size=0.2642921407491152 0.4650757257270274 0.6339946208375731; visual box size=0.2642921407491152 0.4650757257270274 0.6339946208375731
- added link 5, mass 1; collision box size=0.2525206901764938 0.408315794425397 0.5018792704310537; visual box size=0.2525206901764938 0.408315794425397 0.5018792704310537
- added link 6, mass 1; collision box size=0.26060997361750343 0.46621937559833876 0.4351737791623596; visual box size=0.26060997361750343 0.46621937559833876 0.4351737791623596
- added link 7, mass 1; collision box size=0.2944292883272437 0.4778189673426748 0.6615488385795629; visual box size=0.2944292883272437 0.4778189673426748 0.6615488385795629
Joints:
- removed joint Torso_BackLeg
- removed joint Torso_FrontLeg
- added joint 0_1: type revolute, parent 0, child 1, origin xyz=0.2 0 1.5 rpy=0 0 0, axis 0 0 1, limit lower=-3.14159 upper=3.14159 effort=0.0 velocity=0.0
- added joint 1_2: type revolute, parent 1, child 2, origin xyz=0.04627988565601629 0 0.11454886518442267 rpy=0 0 0, axis 1 0 0, limit lower=-3.14159 upper=3.14159 effort=0.0 velocity=0.0
- added joint 2_3: type revolute, parent 2, child 3, origin xyz=0.10772104943893691 0 0.1226297681631432 rpy=0 0 0, axis 1 0 0, limit lower=-3.14159 upper=3.14159 effort=0.0 velocity=0.0
- added joint 3_4: type revolute, parent 3, child 4, origin xyz=0.023615376351609374 0 -0.22109123154650015 rpy=0 0 0, axis 0 0 1, limit lower=-3.14159 upper=3.14159 effort=0.0 velocity=0.0
- added joint 4_5: type revolute, parent 4, child 5, origin xyz=0.0 0.2325378628635137 -0.09590607887228653 rpy=0 0 0, axis 1 0 0, limit lower=-3.14159 upper=3.14159 effort=0.0 velocity=0.0
- added joint 5_6: type revolute, parent 5, child 6, origin xyz=-0.1262603450882469 -0.028379965650815187 0.0 rpy=0 0 0, axis 1 0 0, limit lower=-3.14159 upper=3.14159 effort=0.0 velocity=0.0
- added joint 6_7: type revolute, parent 6, child 7, origin xyz=-0.00404464172050481 0.23310968779916938 0.0 rpy=0 0 0, axis 0 0 1, limit lower=-3.14159 upper=3.14159 effort=0.0 velocity=0.0

Commit message: UGH

File: body.urdf (robot description, URDF)
Before this commit: robot robot, 8 links, 7 joints
Links:
- added link 8, mass 1; collision box size=0.22402606561797472 0.4437401656315195 0.47398246769778346; visual box size=0.22402606561797472 0.4437401656315195 0.47398246769778346
- added link 9, mass 1; collision box size=0.2155493251800286 0.47954892467571747 0.6293992337566363; visual box size=0.2155493251800286 0.47954892467571747 0.6293992337566363
- link 1: geometry collision box size=0.2575820818484914 0.2650338924216289 0.3160097152051494; visual box size=0.2575820818484914 0.2650338924216289 0.3160097152051494
- link 2: geometry collision box size=0.23773197919217978 0.41347891420734506 0.5406483940788026; visual box size=0.23773197919217978 0.41347891420734506 0.5406483940788026
- link 3: geometry collision box size=0.2434426060004437 0.40120767800208035 0.5876740578099057; visual box size=0.2434426060004437 0.40120767800208035 0.5876740578099057
- link 4: geometry collision box size=0.2628495942224618 0.43004273813878735 0.6729691678021489; visual box size=0.2628495942224618 0.43004273813878735 0.6729691678021489
- link 5: geometry collision box size=0.28701097721382485 0.40685251647728116 0.541806938851985; visual box size=0.28701097721382485 0.40685251647728116 0.541806938851985
- link 6: geometry collision box size=0.22023604026113458 0.458514031298351 0.5403871075005825; visual box size=0.22023604026113458 0.458514031298351 0.5403871075005825
- link 7: geometry collision box size=0.2655543369069048 0.47437065043512455 0.6182244807020888; visual box size=0.2655543369069048 0.47437065043512455 0.6182244807020888
Joints:
- added joint 7_8: type revolute, parent 7, child 8, origin xyz=-0.022659148322885098 0.0 0.3091122403510444 rpy=0 0 0, axis 1 0 0, limit lower=-3.14159 upper=3.14159 effort=0.0 velocity=0.0
- added joint 8_9: type revolute, parent 8, child 9, origin xyz=0.0 -0.22187008281575976 0.0 rpy=0 0 0, axis 0 1 0, limit lower=-3.14159 upper=3.14159 effort=0.0 velocity=0.0
- joint 1_2: origin xyz=0.04627988565601629 0 0.11454886518442267 rpy=0 0 0 -> xyz=-0.07120895907575431 0 0.1580048576025747 rpy=0 0 0
- joint 2_3: origin xyz=0.10772104943893691 0 0.1226297681631432 rpy=0 0 0 -> xyz=0.0 -0.20673945710367253 0 rpy=0 0 0
- joint 3_4: axis 0 0 1 -> 1 0 0; origin xyz=0.023615376351609374 0 -0.22109123154650015 rpy=0 0 0 -> xyz=0.12172130300022185 0.006135618102632356 0.11231933943682648 rpy=0 0 0
- joint 4_5: origin xyz=0.0 0.2325378628635137 -0.09590607887228653 rpy=0 0 0 -> xyz=0.00970349411100907 0.21502136906939368 0.0 rpy=0 0 0
- joint 5_6: origin xyz=-0.1262603450882469 -0.028379965650815187 0.0 rpy=0 0 0 -> xyz=0.0 0.19183114740788748 0.0 rpy=0 0 0
- joint 6_7: origin xyz=-0.00404464172050481 0.23310968779916938 0.0 rpy=0 0 0 -> xyz=-0.11011802013056729 0.02583075741053492 0.0 rpy=0 0 0
