Commit message: Progress on assign. 8

File: body0.urdf (robot description, URDF)
Before this commit: robot robot, 3 links, 2 joints
Links:
- link 1: geometry collision box size=0.2608809630808208 0.4235478828817485 0.2528152474023273; visual box size=0.2608809630808208 0.4235478828817485 0.2528152474023273
- link 2: geometry collision box size=0.21175071592489758 0.4505793030617369 0.5174129085328896; visual box size=0.21175071592489758 0.4505793030617369 0.5174129085328896
Joints:
- joint 1_2: origin xyz=0.04167468674850189 -0.11415565155060987 0 rpy=0 0 0 -> xyz=-0.0695595184595896 0 0.12640762370116365 rpy=0 0 0

File: body5.urdf (robot description, URDF)
Before this commit: robot robot, 3 links, 2 joints
Links:
- link 1: geometry collision box size=0.36554655940843495 0.3886724672879093 0.4706912294229822; visual box size=0.36554655940843495 0.3886724672879093 0.4706912294229822
- link 2: geometry collision box size=0.25717775058971143 0.4356887417502669 0.4974867009407369; visual box size=0.25717775058971143 0.4356887417502669 0.4974867009407369
Joints:
- joint 1_2: origin xyz=0.04167468674850189 -0.11415565155060987 0 rpy=0 0 0 -> xyz=0.16554655940843493 0 0.0 rpy=0 0 0

File: body8.urdf (robot description, URDF)
Before this commit: robot robot, 3 links, 2 joints
Links:
- link 1: geometry collision box size=0.2991152001175838 0.4988795984302108 0.2156830186014788; visual box size=0.2991152001175838 0.4988795984302108 0.2156830186014788
- link 2: geometry collision box size=0.28917613100590656 0.46059758313707094 0.5934926264089978; visual box size=0.28917613100590656 0.46059758313707094 0.5934926264089978
Joints:
- joint 1_2: origin xyz=0.04167468674850189 -0.11415565155060987 0 rpy=0 0 0 -> xyz=-0.05044239994120811 0 -0.1078415093007394 rpy=0 0 0

Commit message: Bruh

File: body0.urdf (robot description, URDF)
Before this commit: robot robot, 3 links, 2 joints
Links:
- added link 3, mass 1; collision box size=0.2889732531713186 0.42606700990150187 0.5119025400847931; visual box size=0.2889732531713186 0.42606700990150187 0.5119025400847931
- added link 4, mass 1; collision box size=0.2570472882786366 0.40475828869054037 0.4118727794050135; visual box size=0.2570472882786366 0.40475828869054037 0.4118727794050135
- added link 5, mass 1; collision box size=0.24868399865607807 0.45824658103306126 0.41063936802891987; visual box size=0.24868399865607807 0.45824658103306126 0.41063936802891987
- added link 6, mass 1; collision box size=0.29289408419564356 0.42393333090218527 0.4400851931466311; visual box size=0.29289408419564356 0.42393333090218527 0.4400851931466311
- added link 7, mass 1; collision box size=0.21551426091170586 0.4850884241200714 0.5515412105972993; visual box size=0.21551426091170586 0.4850884241200714 0.5515412105972993
- added link 8, mass 1; collision box size=0.22270895375710315 0.4616983126181626 0.6118676485630552; visual box size=0.22270895375710315 0.4616983126181626 0.6118676485630552
- link 1: geometry collision box size=0.43018350966663715 0.3573689189276218 0.3829607186879096; visual box size=0.43018350966663715 0.3573689189276218 0.3829607186879096
- link 2: geometry collision box size=0.29245234224483674 0.45066758219411135 0.5076111844940331; visual box size=0.29245234224483674 0.45066758219411135 0.5076111844940331
Joints:
- added joint 2_3: type revolute, parent 2, child 3, origin xyz=0.14622617112241837 0 0.06232523290306169 rpy=0 0 0, axis 1 0 0, limit lower=-3.14159 upper=3.14159 effort=0.0 velocity=0.0
- added joint 3_4: type revolute, parent 3, child 4, origin xyz=-0.0017395445367590634 0 -0.25595127004239654 rpy=0 0 0, axis 0 0 1, limit lower=-3.14159 upper=3.14159 effort=0.0 velocity=0.0
- added joint 4_5: type revolute, parent 4, child 5, origin xyz=-0.1285236441393183 0 0.050014880339889656 rpy=0 0 0, axis 0 1 0, limit lower=-3.14159 upper=3.14159 effort=0.0 velocity=0.0
- added joint 5_6: type revolute, parent 5, child 6, origin xyz=-0.12016035451675976 0 0.0 rpy=0 0 0, axis 1 0 0, limit lower=-3.14159 upper=3.14159 effort=0.0 velocity=0.0
- added joint 6_7: type revolute, parent 6, child 7, origin xyz=-0.022105042769782743 0 -0.22004259657331554 rpy=0 0 0, axis 0 1 0, limit lower=-3.14159 upper=3.14159 effort=0.0 velocity=0.0
- added joint 7_8: type revolute, parent 7, child 8, origin xyz=0.10775713045585293 0 -0.05572800872533423 rpy=0 0 0, axis 0 1 0, limit lower=-3.14159 upper=3.14159 effort=0.0 velocity=0.0
- joint 1_2: origin xyz=-0.0695595184595896 0 0.12640762370116365 rpy=0 0 0 -> xyz=0.015091754833318566 0 0.1914803593439548 rpy=0 0 0

File: body1.urdf (robot description, URDF)
Before this commit: robot robot, 6 links, 5 joints
Links:
- removed link 5
- link 1: geometry collision box size=0.24643663760069878 0.48081486394698103 0.479619340255793; visual box size=0.24643663760069878 0.48081486394698103 0.479619340255793
- link 2: geometry collision box size=0.2623150178796507 0.41231767794380897 0.6536262058820654; visual box size=0.2623150178796507 0.41231767794380897 0.6536262058820654
- link 3: geometry collision box size=0.24641310603185887 0.4644805821498851 0.5090712203872099; visual box size=0.24641310603185887 0.4644805821498851 0.5090712203872099
- link 4: geometry collision box size=0.2210541098041285 0.47682005858369275 0.673846600366239; visual box size=0.2210541098041285 0.47682005858369275 0.673846600366239
Joints:
- removed joint 4_5
- joint 1_2: origin xyz=-0.058228050489820604 0.21256126307407064 0.0 rpy=0 0 0 -> xyz=-0.07678168119965062 0 -0.2398096701278965 rpy=0 0 0
- joint 2_3: origin xyz=0.11661009803745974 0.004486743690172684 0.0 rpy=0 0 0 -> xyz=0.13115750893982536 0 -0.08700343281313616 rpy=0 0 0
- joint 3_4: origin xyz=-0.011397547739236513 0.0 0.2596107312700085 rpy=0 0 0 -> xyz=-0.007950955923895942 0.23224029107494254 0.0 rpy=0 0 0

File: body2.urdf (robot description, URDF)
Before this commit: robot robot, 4 links, 3 joints
Links:
- added link 4, mass 1; collision box size=0.27246448115561395 0.41545503982348725 0.48929848083375505; visual box size=0.27246448115561395 0.41545503982348725 0.48929848083375505
- added link 5, mass 1; collision box size=0.23296561504452906 0.4356156801184287 0.5356776778433958; visual box size=0.23296561504452906 0.4356156801184287 0.5356776778433958
- added link 6, mass 1; collision box size=0.2989537278031824 0.4766612612419956 0.5744596490425661; visual box size=0.2989537278031824 0.4766612612419956 0.5744596490425661
- added link 7, mass 1; collision box size=0.24138500567606913 0.425336179226673 0.6110592164887771; visual box size=0.24138500567606913 0.425336179226673 0.6110592164887771
- added link 8, mass 1; collision box size=0.29098987503927026 0.41483722450753896 0.6978712612389961; visual box size=0.29098987503927026 0.41483722450753896 0.6978712612389961
- added link 9, mass 1; collision box size=0.213948299445065 0.4575733734332173 0.5550889758117661; visual box size=0.213948299445065 0.4575733734332173 0.5550889758117661
- link 1: geometry collision box size=0.38996326993169195 0.3096438638432534 0.29142648969454427; visual box size=0.38996326993169195 0.3096438638432534 0.29142648969454427
- link 2: geometry collision box size=0.24463237900352242 0.4734191529405904 0.5229633734821458; visual box size=0.24463237900352242 0.4734191529405904 0.5229633734821458
- link 3: geometry collision box size=0.251105349526791 0.4115346689884266 0.486260731462854; visual box size=0.251105349526791 0.4115346689884266 0.486260731462854
Joints:
- added joint 3_4: type revolute, parent 3, child 4, origin xyz=0.0 -0.03094224197608189 -0.243130365731427 rpy=0 0 0, axis 0 1 0, limit lower=-3.14159 upper=3.14159 effort=0.0 velocity=0.0
- added joint 4_5: type revolute, parent 4, child 5, origin xyz=0.0 -0.20772751991174362 0.0 rpy=0 0 0, axis 0 0 1, limit lower=-3.14159 upper=3.14159 effort=0.0 velocity=0.0
- added joint 5_6: type revolute, parent 5, child 6, origin xyz=0.0 -0.010080320147470734 -0.26935771360714833 rpy=0 0 0, axis 0 0 1, limit lower=-3.14159 upper=3.14159 effort=0.0 velocity=0.0
- added joint 6_7: type revolute, parent 6, child 7, origin xyz=-0.1494768639015912 0.0 -0.019390985599585076 rpy=0 0 0, axis 0 0 1, limit lower=-3.14159 upper=3.14159 effort=0.0 velocity=0.0
- added joint 7_8: type revolute, parent 7, child 8, origin xyz=-0.09190814177447792 0.0 0.0 rpy=0 0 0, axis 1 0 0, limit lower=-3.14159 upper=3.14159 effort=0.0 velocity=0.0
- added joint 8_9: type revolute, parent 8, child 9, origin xyz=-0.024802434681600566 0.0 -0.34893563061949806 rpy=0 0 0, axis 0 0 1, limit lower=-3.14159 upper=3.14159 effort=0.0 velocity=0.0
- joint 1_2: axis 0 0 1 -> 0 1 0; origin xyz=0.015650206697849722 0 0.0 rpy=0 0 0 -> xyz=0.18996326993169194 0 0.0 rpy=0 0 0
- joint 2_3: axis 1 0 0 -> 0 0 1; origin xyz=-0.007807056550349745 0 0.23878641582361726 rpy=0 0 0 -> xyz=-0.07266544546408477 0.2367095764702952 0.0 rpy=0 0 0

File: body3.urdf (robot description, URDF)
Before this commit: robot robot, 11 links, 10 joints
Links:
- removed link 10
- removed link 9
- link 1: geometry collision box size=0.43018350966663715 0.3573689189276218 0.3829607186879096; visual box size=0.43018350966663715 0.3573689189276218 0.3829607186879096
- link 2: geometry collision box size=0.29245234224483674 0.45066758219411135 0.5076111844940331; visual box size=0.29245234224483674 0.45066758219411135 0.5076111844940331
- link 3: geometry collision box size=0.2889732531713186 0.42606700990150187 0.5119025400847931; visual box size=0.2889732531713186 0.42606700990150187 0.5119025400847931
- link 4: geometry collision box size=0.2570472882786366 0.40475828869054037 0.4118727794050135; visual box size=0.2570472882786366 0.40475828869054037 0.4118727794050135
- link 5: geometry collision box size=0.24868399865607807 0.45824658103306126 0.41063936802891987; visual box size=0.24868399865607807 0.45824658103306126 0.41063936802891987
- link 6: geometry collision box size=0.29289408419564356 0.42393333090218527 0.4400851931466311; visual box size=0.29289408419564356 0.42393333090218527 0.4400851931466311
- link 7: geometry collision box size=0.21551426091170586 0.4850884241200714 0.5515412105972993; visual box size=0.21551426091170586 0.4850884241200714 0.5515412105972993
- link 8: geometry collision box size=0.22270895375710315 0.4616983126181626 0.6118676485630552; visual box size=0.22270895375710315 0.4616983126181626 0.6118676485630552
Joints:
- removed joint 8_9
- removed joint 9_10
- joint 1_2: axis 0 0 1 -> 1 0 0; origin xyz=-0.06832538864132595 0 0.11939452628774846 rpy=0 0 0 -> xyz=0.015091754833318566 0 0.1914803593439548 rpy=0 0 0
- joint 2_3: axis 0 1 0 -> 1 0 0; origin xyz=0.0 0 0.28167888742717756 rpy=0 0 0 -> xyz=0.14622617112241837 0 0.06232523290306169 rpy=0 0 0
- joint 3_4: axis 0 1 0 -> 0 0 1; origin xyz=0.0 0 0.21483959079183132 rpy=0 0 0 -> xyz=-0.0017395445367590634 0 -0.25595127004239654 rpy=0 0 0
- joint 4_5: origin xyz=0.0 0.2318506612985579 0.09221822167882898 rpy=0 0 0 -> xyz=-0.1285236441393183 0 0.050014880339889656 rpy=0 0 0
- joint 5_6: axis 0 0 1 -> 1 0 0; origin xyz=0.0 0.235072603343326 0.0 rpy=0 0 0 -> xyz=-0.12016035451675976 0 0.0 rpy=0 0 0
- joint 6_7: origin xyz=0.0 0.015649149163517673 -0.23965034337477895 rpy=0 0 0 -> xyz=-0.022105042769782743 0 -0.22004259657331554 rpy=0 0 0
- joint 7_8: axis 1 0 0 -> 0 1 0; origin xyz=0.11708442718500968 0.0 -0.06401631571358601 rpy=0 0 0 -> xyz=0.10775713045585293 0 -0.05572800872533423 rpy=0 0 0

File: body4.urdf (robot description, URDF)
Before this commit: robot robot, 5 links, 4 joints
Links:
- link 1: geometry collision box size=0.24643663760069878 0.48081486394698103 0.479619340255793; visual box size=0.24643663760069878 0.48081486394698103 0.479619340255793
- link 2: geometry collision box size=0.2623150178796507 0.41231767794380897 0.6536262058820654; visual box size=0.2623150178796507 0.41231767794380897 0.6536262058820654
- link 3: geometry collision box size=0.24641310603185887 0.4644805821498851 0.5090712203872099; visual box size=0.24641310603185887 0.4644805821498851 0.5090712203872099
- link 4: geometry collision box size=0.2210541098041285 0.47682005858369275 0.673846600366239; visual box size=0.2210541098041285 0.47682005858369275 0.673846600366239
Joints:
- joint 1_2: axis 1 0 0 -> 0 0 1; origin xyz=-0.08155151105257245 0.1586342619699342 0.0 rpy=0 0 0 -> xyz=-0.07678168119965062 0 -0.2398096701278965 rpy=0 0 0
- joint 2_3: axis 0 1 0 -> 1 0 0; origin xyz=0.1368109876904389 0.04572848368039026 0.0 rpy=0 0 0 -> xyz=0.13115750893982536 0 -0.08700343281313616 rpy=0 0 0
- joint 3_4: axis 1 0 0 -> 0 1 0; origin xyz=-0.018027249680740542 0.0 -0.261604422351972 rpy=0 0 0 -> xyz=-0.007950955923895942 0.23224029107494254 0.0 rpy=0 0 0

File: body5.urdf (robot description, URDF)
Before this commit: robot robot, 3 links, 2 joints
Links:
- added link 3, mass 1; collision box size=0.251105349526791 0.4115346689884266 0.486260731462854; visual box size=0.251105349526791 0.4115346689884266 0.486260731462854
- added link 4, mass 1; collision box size=0.27246448115561395 0.41545503982348725 0.48929848083375505; visual box size=0.27246448115561395 0.41545503982348725 0.48929848083375505
- added link 5, mass 1; collision box size=0.23296561504452906 0.4356156801184287 0.5356776778433958; visual box size=0.23296561504452906 0.4356156801184287 0.5356776778433958
- added link 6, mass 1; collision box size=0.2989537278031824 0.4766612612419956 0.5744596490425661; visual box size=0.2989537278031824 0.4766612612419956 0.5744596490425661
- added link 7, mass 1; collision box size=0.24138500567606913 0.425336179226673 0.6110592164887771; visual box size=0.24138500567606913 0.425336179226673 0.6110592164887771
- added link 8, mass 1; collision box size=0.29098987503927026 0.41483722450753896 0.6978712612389961; visual box size=0.29098987503927026 0.41483722450753896 0.6978712612389961
- added link 9, mass 1; collision box size=0.213948299445065 0.4575733734332173 0.5550889758117661; visual box size=0.213948299445065 0.4575733734332173 0.5550889758117661
- link 1: geometry collision box size=0.38996326993169195 0.3096438638432534 0.29142648969454427; visual box size=0.38996326993169195 0.3096438638432534 0.29142648969454427
- link 2: geometry collision box size=0.24463237900352242 0.4734191529405904 0.5229633734821458; visual box size=0.24463237900352242 0.4734191529405904 0.5229633734821458
Joints:
- added joint 2_3: type revolute, parent 2, child 3, origin xyz=-0.07266544546408477 0.2367095764702952 0.0 rpy=0 0 0, axis 0 0 1, limit lower=-3.14159 upper=3.14159 effort=0.0 velocity=0.0
- added joint 3_4: type revolute, parent 3, child 4, origin xyz=0.0 -0.03094224197608189 -0.243130365731427 rpy=0 0 0, axis 0 1 0, limit lower=-3.14159 upper=3.14159 effort=0.0 velocity=0.0
- added joint 4_5: type revolute, parent 4, child 5, origin xyz=0.0 -0.20772751991174362 0.0 rpy=0 0 0, axis 0 0 1, limit lower=-3.14159 upper=3.14159 effort=0.0 velocity=0.0
- added joint 5_6: type revolute, parent 5, child 6, origin xyz=0.0 -0.010080320147470734 -0.26935771360714833 rpy=0 0 0, axis 0 0 1, limit lower=-3.14159 upper=3.14159 effort=0.0 velocity=0.0
- added joint 6_7: type revolute, parent 6, child 7, origin xyz=-0.1494768639015912 0.0 -0.019390985599585076 rpy=0 0 0, axis 0 0 1, limit lower=-3.14159 upper=3.14159 effort=0.0 velocity=0.0
- added joint 7_8: type revolute, parent 7, child 8, origin xyz=-0.09190814177447792 0.0 0.0 rpy=0 0 0, axis 1 0 0, limit lower=-3.14159 upper=3.14159 effort=0.0 velocity=0.0
- added joint 8_9: type revolute, parent 8, child 9, origin xyz=-0.024802434681600566 0.0 -0.34893563061949806 rpy=0 0 0, axis 0 0 1, limit lower=-3.14159 upper=3.14159 effort=0.0 velocity=0.0
- joint 1_2: axis 1 0 0 -> 0 1 0; origin xyz=0.16554655940843493 0 0.0 rpy=0 0 0 -> xyz=0.18996326993169194 0 0.0 rpy=0 0 0
