Commit message: Not sure

File: body0.urdf (robot description, URDF)
Before this commit: robot robot, 9 links, 8 joints
Links:
- removed link 6
- removed link 7
- removed link 8
- link 1: geometry collision box size=0.44279752513611936 0.273260133321641 0.3157471717079541; visual box size=0.44279752513611936 0.273260133321641 0.3157471717079541
- link 2: geometry collision box size=0.27042082913154447 0.48468006756385107 0.4489865582670424; visual box size=0.27042082913154447 0.48468006756385107 0.4489865582670424
- link 3: geometry collision box size=0.2612967904610531 0.48027422806237485 0.599303948662542; visual box size=0.2612967904610531 0.48027422806237485 0.599303948662542
- link 4: geometry collision box size=0.23874003598865437 0.46863997927328876 0.518342066095742; visual box size=0.23874003598865437 0.46863997927328876 0.518342066095742
- link 5: geometry collision box size=0.23774604797185073 0.4364557825362556 0.4069128925822804; visual box size=0.23774604797185073 0.4364557825362556 0.4069128925822804
Joints:
- removed joint 5_6
- removed joint 6_7
- removed joint 7_8
- joint 1_2: axis 1 0 0 -> 0 0 1; origin xyz=0.015091754833318566 0 0.1914803593439548 rpy=0 0 0 -> xyz=0.24279752513611935 0 0.0 rpy=0 0 0
- joint 2_3: axis 1 0 0 -> 0 0 1; origin xyz=0.14622617112241837 0 0.06232523290306169 rpy=0 0 0 -> xyz=-0.08618834800228747 0 0.2244932791335212 rpy=0 0 0
- joint 3_4: axis 0 0 1 -> 0 1 0; origin xyz=-0.0017395445367590634 0 -0.25595127004239654 rpy=0 0 0 -> xyz=-0.13064839523052654 0 0.07515869519774987 rpy=0 0 0
- joint 4_5: axis 0 1 0 -> 0 0 1; origin xyz=-0.1285236441393183 0 0.050014880339889656 rpy=0 0 0 -> xyz=0.011278377236199372 0 0.259171033047871 rpy=0 0 0

File: body1.urdf (robot description, URDF)
Before this commit: robot robot, 5 links, 4 joints
Links:
- added link 5, mass 1; collision box size=0.22994927228531806 0.49997777079699324 0.640519612450654; visual box size=0.22994927228531806 0.49997777079699324 0.640519612450654
- added link 6, mass 1; collision box size=0.2506803299654763 0.46922865008247144 0.6886672821462194; visual box size=0.2506803299654763 0.46922865008247144 0.6886672821462194
- added link 7, mass 1; collision box size=0.22984899449118248 0.4766563846903109 0.5892271120761906; visual box size=0.22984899449118248 0.4766563846903109 0.5892271120761906
- link 1: geometry collision box size=0.3880518495190687 0.30620588134074617 0.23123549132827032; visual box size=0.3880518495190687 0.30620588134074617 0.23123549132827032
- link 2: geometry collision box size=0.2120695763602184 0.48288151391958234 0.6671489312329736; visual box size=0.2120695763602184 0.48288151391958234 0.6671489312329736
- link 3: geometry collision box size=0.2151283674965755 0.4632747081351354 0.49275426538891154; visual box size=0.2151283674965755 0.4632747081351354 0.49275426538891154
- link 4: geometry collision box size=0.21667474623389063 0.48119645037526265 0.5444761656691095; visual box size=0.21667474623389063 0.48119645037526265 0.5444761656691095
Joints:
- added joint 4_5: type revolute, parent 4, child 5, origin xyz=-0.0007731893686575703 0.24059822518763133 0.0 rpy=0 0 0, axis 0 1 0, limit lower=-3.14159 upper=3.14159 effort=0.0 velocity=0.0
- added joint 5_6: type revolute, parent 5, child 6, origin xyz=-0.11497463614265903 0.00939066021086532 0.0 rpy=0 0 0, axis 0 1 0, limit lower=-3.14159 upper=3.14159 effort=0.0 velocity=0.0
- added joint 6_7: type revolute, parent 6, child 7, origin xyz=-0.13570569382281727 0.0 0.0 rpy=0 0 0, axis 0 0 1, limit lower=-3.14159 upper=3.14159 effort=0.0 velocity=0.0
- joint 1_2: axis 0 0 1 -> 1 0 0; origin xyz=-0.07678168119965062 0 -0.2398096701278965 rpy=0 0 0 -> xyz=-0.0059740752404656705 0 0.11561774566413516 rpy=0 0 0
- joint 2_3: axis 1 0 0 -> 0 0 1; origin xyz=0.13115750893982536 0 -0.08700343281313616 rpy=0 0 0 -> xyz=0.0 0.24144075695979117 0.21795671995235155 rpy=0 0 0
- joint 3_4: axis 0 1 0 -> 1 0 0; origin xyz=-0.007950955923895942 0.23224029107494254 0.0 rpy=0 0 0 -> xyz=-0.10756418374828774 -0.009803402892223478 0.0 rpy=0 0 0

File: body15.urdf (robot description, URDF)
Before this commit: robot robot, 6 links, 5 joints
Links:
- added link 6, mass 1; collision box size=0.2808720781232919 0.4554224636750253 0.4645391610055529; visual box size=0.2808720781232919 0.4554224636750253 0.4645391610055529
- link 1: geometry collision box size=0.205782564411806 0.23440397607553126 0.43823788877908365; visual box size=0.205782564411806 0.23440397607553126 0.43823788877908365
- link 2: geometry collision box size=0.22956898028687342 0.4861760904635587 0.4206069452899144; visual box size=0.22956898028687342 0.4861760904635587 0.4206069452899144
- link 3: geometry collision box size=0.23728895860891028 0.40804435751073687 0.6179982123604966; visual box size=0.23728895860891028 0.40804435751073687 0.6179982123604966
- link 4: geometry collision box size=0.23772113758391314 0.47375330753999595 0.5851948141454019; visual box size=0.23772113758391314 0.47375330753999595 0.5851948141454019
- link 5: geometry collision box size=0.24125211227057983 0.4018474350034978 0.609335347460261; visual box size=0.24125211227057983 0.4018474350034978 0.609335347460261
Joints:
- added joint 5_6: type revolute, parent 5, child 6, origin xyz=-0.12239154347862326 0.0 0.0 rpy=0 0 0, axis 1 0 0, limit lower=-3.14159 upper=3.14159 effort=0.0 velocity=0.0
- joint 1_2: axis 1 0 0 -> 0 0 1; origin xyz=-0.049374282331946406 -0.2469769683730429 0 rpy=0 0 0 -> xyz=-0.09710871779409701 -0.11720198803776563 0 rpy=0 0 0
- joint 2_3: axis 0 0 1 -> 0 1 0; origin xyz=0.12632669080646872 0.040249193952108436 0.0 rpy=0 0 0 -> xyz=0.0 -0.12588605719401372 0.2103034726449572 rpy=0 0 0
- joint 3_4: axis 0 1 0 -> 0 0 1; origin xyz=0.001088012218124268 0.0 0.32267572418387985 rpy=0 0 0 -> xyz=0.0 0.0 0.4076947397155394 rpy=0 0 0
- joint 4_5: axis 0 0 1 -> 0 1 0; origin xyz=-0.12216043794042813 0.0 -0.10151340072737125 rpy=0 0 0 -> xyz=-0.11886056879195657 0.0 -0.016401699107547074 rpy=0 0 0

File: body16.urdf (robot description, URDF)
Before this commit: robot robot, 11 links, 10 joints
Links:
- removed link 10
- link 1: geometry collision box size=0.3854398360685128 0.3486440392806881 0.3519142537088832; visual box size=0.3854398360685128 0.3486440392806881 0.3519142537088832
- link 2: geometry collision box size=0.25736565630099384 0.4901029859428795 0.5846955122617915; visual box size=0.25736565630099384 0.4901029859428795 0.5846955122617915
- link 3: geometry collision box size=0.24739795004017112 0.49342376578140024 0.654230085626131; visual box size=0.24739795004017112 0.49342376578140024 0.654230085626131
- link 4: geometry collision box size=0.2743621011147051 0.4427224995613169 0.44075183818327857; visual box size=0.2743621011147051 0.4427224995613169 0.44075183818327857
- link 5: geometry collision box size=0.2807215717557156 0.48072516302213786 0.6267848400560464; visual box size=0.2807215717557156 0.48072516302213786 0.6267848400560464
- link 6: geometry collision box size=0.2195766086099828 0.45248558607217987 0.5915732558227198; visual box size=0.2195766086099828 0.45248558607217987 0.5915732558227198
- link 7: geometry collision box size=0.23955310253662485 0.41874565448820233 0.4494619940891822; visual box size=0.23955310253662485 0.41874565448820233 0.4494619940891822
- link 8: geometry collision box size=0.2795004898635607 0.4823652027060712 0.6968948614967263; visual box size=0.2795004898635607 0.4823652027060712 0.6968948614967263
- link 9: geometry collision box size=0.2748060075300834 0.40502061632281755 0.41316268184032556; visual box size=0.2748060075300834 0.40502061632281755 0.41316268184032556
Joints:
- removed joint 9_10
- joint 1_2: axis 0 0 1 -> 0 1 0; origin xyz=0.03480763173296145 0 0.1229019374111993 rpy=0 0 0 -> xyz=-0.007280081965743618 0 0.1759571268544416 rpy=0 0 0
- joint 2_3: axis 1 0 0 -> 0 1 0; origin xyz=0.14035715371600443 0 0.13809437087807996 rpy=0 0 0 -> xyz=0.12868282815049692 0 0.11639062927645427 rpy=0 0 0
- joint 3_4: origin xyz=-0.014835921681921382 -0.2088385233166858 0 rpy=0 0 0 -> xyz=0.11871512188967423 0 0.0 rpy=0 0 0
- joint 4_5: axis 0 1 0 -> 0 0 1; origin xyz=0.1278902120736175 -0.001615034869155485 0.0 rpy=0 0 0 -> xyz=0.013482075537266991 -0.22136124978065844 0 rpy=0 0 0
- joint 5_6: axis 1 0 0 -> 0 0 1; origin xyz=0.019675730094719124 0.24132705051651518 0.0 rpy=0 0 0 -> xyz=-0.1403607858778578 -0.019001331730410492 0.0 rpy=0 0 0
- joint 6_7: axis 1 0 0 -> 0 1 0; origin xyz=0.0 -0.0398124472071556 -0.2718885871860983 rpy=0 0 0 -> xyz=0.030572481572866406 0.22624279303608993 0.0 rpy=0 0 0
- joint 7_8: axis 0 0 1 -> 1 0 0; origin xyz=0.10481175301980657 0.0 -0.022039019320145403 rpy=0 0 0 -> xyz=0.0 -0.016869965791988767 0.2247309970445911 rpy=0 0 0
- joint 8_9: axis 0 1 0 -> 1 0 0; origin xyz=0.03924718123776283 0.2239834935945577 0.0 rpy=0 0 0 -> xyz=0.0 0.2411826013530356 0.12371643370377194 rpy=0 0 0

File: body17.urdf (robot description, URDF)
Before this commit: robot robot, 11 links, 10 joints
Links:
- removed link 10
- link 1: geometry collision box size=0.25082495649509534 0.23073722574166464 0.3064739595049518; visual box size=0.25082495649509534 0.23073722574166464 0.3064739595049518
- link 2: geometry collision box size=0.2658297845588434 0.49996600926991547 0.5442018500203; visual box size=0.2658297845588434 0.49996600926991547 0.5442018500203
- link 3: geometry collision box size=0.22117546699061585 0.4763553098958057 0.48300398895401897; visual box size=0.22117546699061585 0.4763553098958057 0.48300398895401897
- link 4: geometry collision box size=0.21424143978407945 0.4474665716273848 0.4273826111552768; visual box size=0.21424143978407945 0.4474665716273848 0.4273826111552768
- link 5: geometry collision box size=0.2488361006769117 0.43791097623791897 0.40003755228501986; visual box size=0.2488361006769117 0.43791097623791897 0.40003755228501986
- link 6: geometry collision box size=0.23129203336212342 0.4262987924608559 0.5408244753066019; visual box size=0.23129203336212342 0.4262987924608559 0.5408244753066019
- link 7: geometry collision box size=0.262780802483842 0.4361585365666487 0.4621045623613202; visual box size=0.262780802483842 0.4361585365666487 0.4621045623613202
- link 8: geometry collision box size=0.24509096417542764 0.495510408451492 0.6837250061172832; visual box size=0.24509096417542764 0.495510408451492 0.6837250061172832
- link 9: geometry collision box size=0.23168094308105452 0.4275912560057105 0.5969889258117425; visual box size=0.23168094308105452 0.4275912560057105 0.5969889258117425
Joints:
- removed joint 9_10
- joint 1_2: axis 0 0 1 -> 1 0 0; origin xyz=0.03480763173296145 0 0.1229019374111993 rpy=0 0 0 -> xyz=0.05082495649509533 0 0.0 rpy=0 0 0
- joint 2_3: axis 1 0 0 -> 0 0 1; origin xyz=0.14035715371600443 0 0.13809437087807996 rpy=0 0 0 -> xyz=0.1404173063112957 0 0.0 rpy=0 0 0
- joint 3_4: axis 0 1 0 -> 1 0 0; origin xyz=-0.014835921681921382 -0.2088385233166858 0 rpy=0 0 0 -> xyz=0.08826057471119414 0 0.0 rpy=0 0 0
- joint 4_5: axis 0 1 0 -> 1 0 0; origin xyz=0.1278902120736175 -0.001615034869155485 0.0 rpy=0 0 0 -> xyz=-0.003467013603268232 0.2237332858136924 0.0 rpy=0 0 0
- joint 5_6: axis 1 0 0 -> 0 1 0; origin xyz=0.019675730094719124 0.24132705051651518 0.0 rpy=0 0 0 -> xyz=-0.12441805033845585 -0.00477779769473291 0.0 rpy=0 0 0
- joint 6_7: origin xyz=0.0 -0.0398124472071556 -0.2718885871860983 rpy=0 0 0 -> xyz=0.008772033657394152 0.0 0.27041223765330097 rpy=0 0 0
- joint 7_8: axis 0 0 1 -> 0 1 0; origin xyz=0.10481175301980657 0.0 -0.022039019320145403 rpy=0 0 0 -> xyz=0.0 -0.21807926828332436 0.0 rpy=0 0 0
- joint 8_9: axis 0 1 0 -> 1 0 0; origin xyz=0.03924718123776283 0.2239834935945577 0.0 rpy=0 0 0 -> xyz=0.12254548208771382 -0.029675935942421655 -0.03935995647264079 rpy=0 0 0

File: body6.urdf (robot description, URDF)
Before this commit: robot robot, 10 links, 9 joints
Links:
- removed link 5
- removed link 6
- removed link 7
- removed link 8
- removed link 9
- link 1: geometry collision box size=0.22369200198265848 0.3125225110186299 0.3389517249237382; visual box size=0.22369200198265848 0.3125225110186299 0.3389517249237382
- link 2: geometry collision box size=0.21855222535414928 0.4544429512685429 0.44569976516772075; visual box size=0.21855222535414928 0.4544429512685429 0.44569976516772075
- link 3: geometry collision box size=0.26064695316694875 0.4265465975519118 0.4994731785157402; visual box size=0.26064695316694875 0.4265465975519118 0.4994731785157402
- link 4: geometry collision box size=0.25413855140362185 0.4274113575020218 0.5213076620148622; visual box size=0.25413855140362185 0.4274113575020218 0.5213076620148622
Joints:
- removed joint 4_5
- removed joint 5_6
- removed joint 6_7
- removed joint 7_8
- removed joint 8_9
- joint 1_2: axis 0 1 0 -> 1 0 0; origin xyz=0.006770270251041072 0 0.13896686500556596 rpy=0 0 0 -> xyz=-0.08815399900867077 0 0.1694758624618691 rpy=0 0 0
- joint 2_3: axis 0 1 0 -> 1 0 0; origin xyz=0.0 0 0.2720008308990989 rpy=0 0 0 -> xyz=-0.10927611267707464 0 0.05337402012199122 rpy=0 0 0
- joint 3_4: axis 0 0 1 -> 1 0 0; origin xyz=0.10534989888042448 0 0.0974797142324988 rpy=0 0 0 -> xyz=-0.021047363906399733 0.2132732987759559 0.0 rpy=0 0 0

File: body7.urdf (robot description, URDF)
Before this commit: robot robot, 7 links, 6 joints
Links:
- removed link 5
- removed link 6
- link 1: geometry collision box size=0.24385207838929915 0.27594847781084214 0.24819210165493052; visual box size=0.24385207838929915 0.27594847781084214 0.24819210165493052
- link 2: geometry collision box size=0.2868335090493649 0.43282813291781813 0.6468591912649794; visual box size=0.2868335090493649 0.43282813291781813 0.6468591912649794
- link 3: geometry collision box size=0.22083077622824382 0.4208701876648332 0.646325005459937; visual box size=0.22083077622824382 0.4208701876648332 0.646325005459937
- link 4: geometry collision box size=0.274343312811756 0.48291650949186 0.5028915748972227; visual box size=0.274343312811756 0.48291650949186 0.5028915748972227
Joints:
- removed joint 4_5
- removed joint 5_6
- joint 1_2: axis 1 0 0 -> 0 1 0; origin xyz=0.040575950015197176 -0.1956625762093365 0 rpy=0 0 0 -> xyz=-0.07807396080535044 -0.13797423890542107 0 rpy=0 0 0
- joint 2_3: axis 0 0 1 -> 0 1 0; origin xyz=-0.10001305080853634 -0.012349531712785966 0.0 rpy=0 0 0 -> xyz=0.0 -0.078439827553488 0.3234295956324897 rpy=0 0 0
- joint 3_4: axis 0 1 0 -> 0 0 1; origin xyz=-0.04388887703060851 0.230284412220578 0.0 rpy=0 0 0 -> xyz=-0.11041538811412191 0.0 -0.00026709290252124873 rpy=0 0 0

File: body8.urdf (robot description, URDF)
Before this commit: robot robot, 3 links, 2 joints
Links:
- added link 3, mass 1; collision box size=0.25482940604918597 0.4423744894224681 0.6453514483677597; visual box size=0.25482940604918597 0.4423744894224681 0.6453514483677597
- added link 4, mass 1; collision box size=0.24432087588085627 0.4247176264061547 0.4423246469130172; visual box size=0.24432087588085627 0.4247176264061547 0.4423246469130172
- added link 5, mass 1; collision box size=0.23146353959832433 0.4399616972047096 0.42316336682429173; visual box size=0.23146353959832433 0.4399616972047096 0.42316336682429173
- link 1: geometry collision box size=0.3012514353361072 0.4939539367460858 0.41158777515972034; visual box size=0.3012514353361072 0.4939539367460858 0.41158777515972034
- link 2: geometry collision box size=0.25265338161293743 0.4134555488418689 0.5804052840804795; visual box size=0.25265338161293743 0.4134555488418689 0.5804052840804795
Joints:
- added joint 2_3: type revolute, parent 2, child 3, origin xyz=0.12632669080646872 0.040249193952108436 0.0 rpy=0 0 0, axis 0 0 1, limit lower=-3.14159 upper=3.14159 effort=0.0 velocity=0.0
- added joint 3_4: type revolute, parent 3, child 4, origin xyz=0.001088012218124268 0.0 0.32267572418387985 rpy=0 0 0, axis 0 1 0, limit lower=-3.14159 upper=3.14159 effort=0.0 velocity=0.0
- added joint 4_5: type revolute, parent 4, child 5, origin xyz=-0.12216043794042813 0.0 -0.10151340072737125 rpy=0 0 0, axis 0 0 1, limit lower=-3.14159 upper=3.14159 effort=0.0 velocity=0.0
- joint 1_2: origin xyz=-0.05044239994120811 0 -0.1078415093007394 rpy=0 0 0 -> xyz=-0.049374282331946406 -0.2469769683730429 0 rpy=0 0 0

File: body9.urdf (robot description, URDF)
Before this commit: robot robot, 9 links, 8 joints
Links:
- removed link 5
- removed link 6
- removed link 7
- removed link 8
- link 1: geometry collision box size=0.22369200198265848 0.3125225110186299 0.3389517249237382; visual box size=0.22369200198265848 0.3125225110186299 0.3389517249237382
- link 2: geometry collision box size=0.21855222535414928 0.4544429512685429 0.44569976516772075; visual box size=0.21855222535414928 0.4544429512685429 0.44569976516772075
- link 3: geometry collision box size=0.26064695316694875 0.4265465975519118 0.4994731785157402; visual box size=0.26064695316694875 0.4265465975519118 0.4994731785157402
- link 4: geometry collision box size=0.25413855140362185 0.4274113575020218 0.5213076620148622; visual box size=0.25413855140362185 0.4274113575020218 0.5213076620148622
Joints:
- removed joint 4_5
- removed joint 5_6
- removed joint 6_7
- removed joint 7_8
- joint 1_2: axis 0 1 0 -> 1 0 0; origin xyz=0.027077026152469014 0.21898474299132004 0.0 rpy=0 0 0 -> xyz=-0.08815399900867077 0 0.1694758624618691 rpy=0 0 0
- joint 2_3: axis 0 1 0 -> 1 0 0; origin xyz=0.10929965068832725 -0.017930313681351617 0.0 rpy=0 0 0 -> xyz=-0.10927611267707464 0 0.05337402012199122 rpy=0 0 0
- joint 3_4: axis 0 1 0 -> 1 0 0; origin xyz=0.032633202747796575 0.0 0.23533786693450257 rpy=0 0 0 -> xyz=-0.021047363906399733 0.2132732987759559 0.0 rpy=0 0 0
